Commit message: modifications for Lindsey: change camera name, change obstacle layer parameters, change chest camera model

File: strands_description/urdf/scitos_all_robot_model.xacro (robot description, xacro)
@@ -9,5 +9,5 @@
   <xacro:include filename="$(find scitos_description)/urdf/scitos.xacro" />
   <!-- Connect base to chest_xtion_link -->
-  <link name="chest_xtion_link">
+  <link name="chest_rs_link">
     <visual>
       <origin rpy="3.14 0 0" xyz="0 0 0"/>
@@ -23,48 +23,19 @@
     </collision>
   </link>
-  <link name="chest_xtion_height_tilt_link"/>
-  <joint name="chest_xtion_height_joint" type="prismatic" >
+  <link name="chest_rs_height_tilt_link"/>
+  <joint name="chest_rs_height_joint" type="prismatic" >
     <!-- Z height from calibrate_chest -->
-    <axis xyz="0 0 1"/>
-    <origin rpy="0 0 0" xyz="0.0294 0 0" />
+    <axis xyz="0 0 0"/>
+    <origin rpy="0 0 0" xyz="0.0294 0 1.163665" />
     <limit effort="1000" velocity="1000" lower="0.5" upper="1.5"/>
     <parent link="base_link"/>
-    <child link="chest_xtion_height_tilt_link"/>
+    <child link="chest_rs_height_tilt_link"/>
   </joint>
-  <joint name="chest_xtion_tilt_joint" type="continuous" >
+  <joint name="chest_rs_tilt_joint" type="continuous" >
     <!-- Rotation y angle from calibrate_chest-->
-    <axis xyz="0 1 0"/>
-    <origin rpy="0 0 0" xyz="0 0 0" />
-    <parent link="chest_xtion_height_tilt_link"/>
-    <child link="chest_xtion_link"/>
-  </joint>
-  <!-- chest_xtion internal frames -->
-  <link name="chest_xtion_depth_frame"/>
-  <link name="chest_xtion_rgb_frame"/>
-  <link name="chest_xtion_depth_optical_frame"/>
-  <link name="chest_xtion_rgb_optical_frame"/>
-  <joint name="chest_xtion_base_link" type="fixed" >
-    <origin rpy="0 0 0"
-            xyz="0 0.045 0" />
-    <parent link="chest_xtion_link"/>
-    <child link="chest_xtion_depth_frame"/>
-  </joint>
-  <joint name="chest_xtion_base_link1" type="fixed" >
-    <origin rpy="0 0 0"
-            xyz="0 0.02 0" />
-    <parent link="chest_xtion_link"/>
-    <child link="chest_xtion_rgb_frame"/>
-  </joint>
-  <joint name="chest_xtion_base_link2" type="fixed" >
-    <origin rpy="-1.5707963267948966 0 -1.5707963267948966"
-            xyz="0 0 0" />
-    <parent link="chest_xtion_depth_frame"/>
-    <child link="chest_xtion_depth_optical_frame"/>
-  </joint>
-  <joint name="chest_xtion_base_link3" type="fixed" >
-    <origin rpy="-1.5707963267948966 0 -1.5707963267948966"
-            xyz="0 0 0" />
-    <parent link="chest_xtion_rgb_frame"/>
-    <child link="chest_xtion_rgb_optical_frame"/>
+    <axis xyz="0 0 0"/>
+    <origin rpy="0 0 0.811891" xyz="0 0 0" />
+    <parent link="chest_rs_height_tilt_link"/>
+    <child link="chest_rs_link"/>
   </joint>
 </robot>

File: strands_description/urdf/scitos_chest_camera.xacro (robot description, xacro)
@@ -9,6 +9,6 @@
   <!-- <xacro:include filename="$(find scitos_description)/urdf/scitos_calibration.xacro" /> -->
   <link name="base_link" />
-  <!-- Connect base to chest_xtion_link -->
-  <link name="chest_xtion_link">
+  <!-- Connect base to chest_rs_link -->
+  <link name="chest_rs_link">
     <visual>
       <origin rpy="3.14 0 0" xyz="0 0 0"/>
@@ -24,48 +24,19 @@
     </collision>
   </link>
-  <link name="chest_xtion_height_tilt_link"/>
-  <joint name="chest_xtion_height_joint" type="prismatic" >
+  <link name="chest_rs_height_tilt_link"/>
+  <joint name="chest_rs_height_joint" type="fixed" >
     <!-- Z height from calibrate_chest -->
-    <axis xyz="0 0 1"/>
-    <origin rpy="0 0 0" xyz="0.0294 0 0" />
+    <axis xyz="1 0 0"/>
+    <origin rpy="0 0 0" xyz="0.0294 0 1.161783" />
     <limit effort="1000" velocity="1000" lower="0.5" upper="1.5"/>
     <parent link="base_link"/>
-    <child link="chest_xtion_height_tilt_link"/>
+    <child link="chest_rs_height_tilt_link"/>
   </joint>
-  <joint name="chest_xtion_tilt_joint" type="continuous" >
+  <joint name="chest_rs_tilt_joint" type="fixed" >
     <!-- Rotation y angle from calibrate_chest-->
-    <axis xyz="0 1 0"/>
-    <origin rpy="0 0 0" xyz="0 0 0" />
-    <parent link="chest_xtion_height_tilt_link"/>
-    <child link="chest_xtion_link"/>
-  </joint>
-  <!-- chest_xtion internal frames -->
-  <link name="chest_xtion_depth_frame"/>
-  <link name="chest_xtion_rgb_frame"/>
-  <link name="chest_xtion_depth_optical_frame"/>
-  <link name="chest_xtion_rgb_optical_frame"/>
-  <joint name="chest_xtion_base_link" type="fixed" >
-    <origin rpy="0 0 0"
-            xyz="0 0.045 0" />
-    <parent link="chest_xtion_link"/>
-    <child link="chest_xtion_depth_frame"/>
-  </joint>
-  <joint name="chest_xtion_base_link1" type="fixed" >
-    <origin rpy="0 0 0"
-            xyz="0 0.02 0" />
-    <parent link="chest_xtion_link"/>
-    <child link="chest_xtion_rgb_frame"/>
-  </joint>
-  <joint name="chest_xtion_base_link2" type="fixed" >
-    <origin rpy="-1.5707963267948966 0 -1.5707963267948966"
-            xyz="0 0 0" />
-    <parent link="chest_xtion_depth_frame"/>
-    <child link="chest_xtion_depth_optical_frame"/>
-  </joint>
-  <joint name="chest_xtion_base_link3" type="fixed" >
-    <origin rpy="-1.5707963267948966 0 -1.5707963267948966"
-            xyz="0 0 0" />
-    <parent link="chest_xtion_rgb_frame"/>
-    <child link="chest_xtion_rgb_optical_frame"/>
+    <axis xyz="1 0 0"/>
+    <origin rpy="0 0.862981 0" xyz="0 0 0" />
+    <parent link="chest_rs_height_tilt_link"/>
+    <child link="chest_rs_link"/>
   </joint>
 </robot>

Commit message: putting camera specific things into parameters

File: strands_description/urdf/scitos_all_robot_model.xacro (robot description, xacro)
@@ -9,5 +9,5 @@
   <xacro:include filename="$(find scitos_description)/urdf/scitos.xacro" />
   <!-- Connect base to chest_xtion_link -->
-  <link name="chest_rs_link">
+  <link name="$(arg chest_camera_name)_link">
     <visual>
       <origin rpy="3.14 0 0" xyz="0 0 0"/>
@@ -23,6 +23,6 @@
     </collision>
   </link>
-  <link name="chest_rs_height_tilt_link"/>
-  <joint name="chest_rs_height_joint" type="prismatic" >
+  <link name="$(arg chest_camera_name)_height_tilt_link"/>
+  <joint name="$(arg chest_camera_name)_height_joint" type="prismatic" >
     <!-- Z height from calibrate_chest -->
     <axis xyz="0 0 0"/>
@@ -30,12 +30,44 @@
     <limit effort="1000" velocity="1000" lower="0.5" upper="1.5"/>
     <parent link="base_link"/>
-    <child link="chest_rs_height_tilt_link"/>
+    <child link="$(arg chest_camera_name)_height_tilt_link"/>
   </joint>
-  <joint name="chest_rs_tilt_joint" type="continuous" >
+  <joint name="$(arg chest_camera_name)_tilt_joint" type="continuous" >
     <!-- Rotation y angle from calibrate_chest-->
     <axis xyz="0 0 0"/>
     <origin rpy="0 0 0.811891" xyz="0 0 0" />
-    <parent link="chest_rs_height_tilt_link"/>
-    <child link="chest_rs_link"/>
+    <parent link="$(arg chest_camera_name)_height_tilt_link"/>
+    <child link="$(arg chest_camera_name)_link"/>
   </joint>
+  <xacro:property name="chest_camera_name" value="$(arg chest_camera_name)"/>
+  <xacro:if value="${chest_camera_name == 'chest_xtion'}">
+    <!-- chest_xtion internal frames -->
+    <link name="$(arg chest_camera_name)_depth_frame"/>
+    <link name="$(arg chest_camera_name)_rgb_frame"/>
+    <link name="$(arg chest_camera_name)_depth_optical_frame"/>
+    <link name="$(arg chest_camera_name)_rgb_optical_frame"/>
+    <joint name="$(arg chest_camera_name)_base_link" type="fixed" >
+      <origin rpy="0 0 0"
+            xyz="0 0.045 0" />
+      <parent link="$(arg chest_camera_name)_link"/>
+      <child link="$(arg chest_camera_name)_depth_frame"/>
+    </joint>
+    <joint name="$(arg chest_camera_name)_base_link1" type="fixed" >
+      <origin rpy="0 0 0"
+            xyz="0 0.02 0" />
+      <parent link="$(arg chest_camera_name)_link"/>
+      <child link="$(arg chest_camera_name)_rgb_frame"/>
+    </joint>
+    <joint name="$(arg chest_camera_name)_base_link2" type="fixed" >
+    <origin rpy="-1.5707963267948966 0 -1.5707963267948966"
+            xyz="0 0 0" />
+    <parent link="$(arg chest_camera_name)_depth_frame"/>
+      <child link="$(arg chest_camera_name)_depth_optical_frame"/>
+    </joint>
+    <joint name="$(arg chest_camera_name)_base_link3" type="fixed" >
+      <origin rpy="-1.5707963267948966 0 -1.5707963267948966"
+            xyz="0 0 0" />
+      <parent link="$(arg chest_camera_name)_rgb_frame"/>
+      <child link="$(arg chest_camera_name)_rgb_optical_frame"/>
+    </joint>
+  </xacro:if>
 </robot>

File: strands_description/urdf/scitos_chest_camera.xacro (robot description, xacro)
@@ -10,5 +10,5 @@
   <link name="base_link" />
   <!-- Connect base to chest_rs_link -->
-  <link name="chest_rs_link">
+  <link name="$(arg chest_camera_name)_link">
     <visual>
       <origin rpy="3.14 0 0" xyz="0 0 0"/>
@@ -24,6 +24,6 @@
     </collision>
   </link>
-  <link name="chest_rs_height_tilt_link"/>
-  <joint name="chest_rs_height_joint" type="fixed" >
+  <link name="$(arg chest_camera_name)_height_tilt_link"/>
+  <joint name="$(arg chest_camera_name)_height_joint" type="fixed" >
     <!-- Z height from calibrate_chest -->
     <axis xyz="1 0 0"/>
@@ -31,12 +31,44 @@
     <limit effort="1000" velocity="1000" lower="0.5" upper="1.5"/>
     <parent link="base_link"/>
-    <child link="chest_rs_height_tilt_link"/>
+    <child link="$(arg chest_camera_name)_height_tilt_link"/>
   </joint>
-  <joint name="chest_rs_tilt_joint" type="fixed" >
+  <joint name="$(arg chest_camera_name)_tilt_joint" type="fixed" >
     <!-- Rotation y angle from calibrate_chest-->
     <axis xyz="1 0 0"/>
     <origin rpy="0 0.862981 0" xyz="0 0 0" />
-    <parent link="chest_rs_height_tilt_link"/>
-    <child link="chest_rs_link"/>
+    <parent link="$(arg chest_camera_name)_height_tilt_link"/>
+    <child link="$(arg chest_camera_name)_link"/>
   </joint>
+  <xacro:property name="chest_camera_name" value="$(arg chest_camera_name)"/>
+  <xacro:if value="${chest_camera_name == 'chest_xtion'}">
+    <!-- chest_xtion internal frames -->
+    <link name="$(arg chest_camera_name)_depth_frame"/>
+    <link name="$(arg chest_camera_name)_rgb_frame"/>
+    <link name="$(arg chest_camera_name)_depth_optical_frame"/>
+    <link name="$(arg chest_camera_name)_rgb_optical_frame"/>
+    <joint name="$(arg chest_camera_name)_base_link" type="fixed" >
+      <origin rpy="0 0 0"
+            xyz="0 0.045 0" />
+      <parent link="$(arg chest_camera_name)_link"/>
+      <child link="$(arg chest_camera_name)_depth_frame"/>
+    </joint>
+    <joint name="$(arg chest_camera_name)_base_link1" type="fixed" >
+      <origin rpy="0 0 0"
+            xyz="0 0.02 0" />
+      <parent link="$(arg chest_camera_name)_link"/>
+      <child link="$(arg chest_camera_name)_rgb_frame"/>
+    </joint>
+    <joint name="$(arg chest_camera_name)_base_link2" type="fixed" >
+    <origin rpy="-1.5707963267948966 0 -1.5707963267948966"
+            xyz="0 0 0" />
+    <parent link="$(arg chest_camera_name)_depth_frame"/>
+      <child link="$(arg chest_camera_name)_depth_optical_frame"/>
+    </joint>
+    <joint name="$(arg chest_camera_name)_base_link3" type="fixed" >
+      <origin rpy="-1.5707963267948966 0 -1.5707963267948966"
+            xyz="0 0 0" />
+      <parent link="$(arg chest_camera_name)_rgb_frame"/>
+      <child link="$(arg chest_camera_name)_rgb_optical_frame"/>
+    </joint>
+  </xacro:if>
 </robot>

Commit message: modifications at the museum

File: strands_description/urdf/scitos_all_robot_model.xacro (robot description, xacro)
@@ -35,5 +35,5 @@
     <!-- Rotation y angle from calibrate_chest-->
     <axis xyz="0 0 0"/>
-    <origin rpy="0 0 0.811891" xyz="0 0 0" />
+    <origin rpy="0 0 0.927019" xyz="0 0 0" />
     <parent link="$(arg chest_camera_name)_height_tilt_link"/>
     <child link="$(arg chest_camera_name)_link"/>

File: strands_description/urdf/scitos_chest_camera.xacro (robot description, xacro)
@@ -28,5 +28,5 @@
     <!-- Z height from calibrate_chest -->
     <axis xyz="1 0 0"/>
-    <origin rpy="0 0 0" xyz="0.0294 0 1.161783" />
+    <origin rpy="0 0 0" xyz="0.0294 0 1.16" />
     <limit effort="1000" velocity="1000" lower="0.5" upper="1.5"/>
     <parent link="base_link"/>
@@ -36,5 +36,5 @@
     <!-- Rotation y angle from calibrate_chest-->
     <axis xyz="1 0 0"/>
-    <origin rpy="0 0.862981 0" xyz="0 0 0" />
+    <origin rpy="0 0.85 0" xyz="0 0 0" />
     <parent link="$(arg chest_camera_name)_height_tilt_link"/>
     <child link="$(arg chest_camera_name)_link"/>
